File: hardware/noise_floor.kicad_pcb (KiCad board)
At the start: 2 copper layers, 46 x 115.8 mm, 33 parts, among them J1 DC Power, J10 IO/Switch Connector 1 (Switch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, J11 IO/Switch Connector 2 (Switch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, J2 Input, J3 Output, J4 UX1, J5 UX2, J6 Battery, J7 IO/Effect Connector 1 (IO Sid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, J8 IO/Switch Connector 1 (IO Sid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, J9 IO/Switch Connector 2 (IO Sid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, SW1 Footswitch, SW2 SPDT1, SW3 SPDT2, SW4 SPDT3

Commit message: Further iteration on UX board:
 - Change to square body pots and bump count to six
 - Change to 25-pin board-to-board connectors (and improve footprint)
 - Change optional pot adjustment to 1206 smt resistors
 - Update layout/routing to suit
Parts:
- added R11: 0, Resistor_SMD:R_1206_3216Metric_Pad1.30x1.75mm_HandSolder, F.Cu at (41.0, 113.3)
- added R13: 0, Resistor_SMD:R_1206_3216Metric_Pad1.30x1.75mm_HandSolder, F.Cu at (39.5, 109.7)
- added R15: 0, Resistor_SMD:R_1206_3216Metric_Pad1.30x1.75mm_HandSolder, F.Cu at (25.9, 109.7)
- added R17: 0, Resistor_SMD:R_1206_3216Metric_Pad1.30x1.75mm_HandSolder, F.Cu at (24.4, 113.3)
- added R2: 0, Resistor_SMD:R_1206_3216Metric_Pad1.30x1.75mm_HandSolder, F.Cu at (59.1, 109.7)
- added R20: 0, Resistor_SMD:R_1206_3216Metric_Pad1.30x1.75mm_HandSolder, F.Cu at (22.9, 109.7)
- added R4: 0, Resistor_SMD:R_1206_3216Metric_Pad1.30x1.75mm_HandSolder, F.Cu at (57.6, 113.3)
- added R7: 0, Resistor_SMD:R_1206_3216Metric_Pad1.30x1.75mm_HandSolder, F.Cu at (56.0, 109.7)
- added R9: 0, Resistor_SMD:R_1206_3216Metric_Pad1.30x1.75mm_HandSolder, F.Cu at (42.5, 109.7)
- added RV2: POT4, noise_floor:Potentiometer_Alpha_RD901F-40-00D_Single_Vertical_with_3DModel_from_Vasily_Kashirin, B.Cu at (60.1, 115.3)
- added RV4: POT5, noise_floor:Potentiometer_Alpha_RD901F-40-00D_Single_Vertical_with_3DModel_from_Vasily_Kashirin, B.Cu at (43.5, 115.3)
- added RV6: POT6, noise_floor:Potentiometer_Alpha_RD901F-40-00D_Single_Vertical_with_3DModel_from_Vasily_Kashirin, B.Cu at (26.9, 115.3)
- J11: renamed from J5; footprint noise_floor:Amphenol_Receptacle_15pin_10162581-3134115LF -> noise_floor:Amphenol_Receptacle_25pin_10162581-3134125LF
- J4: footprint noise_floor:Amphenol_Receptacle_15pin_10162581-3134115LF -> noise_floor:Amphenol_Receptacle_25pin_10162581-3134125LF
- R1: footprint Resistor_THT:R_Axial_DIN0207_L6.3mm_D2.5mm_P7.62mm_Horizontal -> Resistor_SMD:R_1206_3216Metric_Pad1.30x1.75mm_HandSolder
- R10: renamed from R9; footprint Resistor_THT:R_Axial_DIN0207_L6.3mm_D2.5mm_P7.62mm_Horizontal -> Resistor_SMD:R_1206_3216Metric_Pad1.30x1.75mm_HandSolder
- R12: renamed from R10; footprint Resistor_THT:R_Axial_DIN0207_L6.3mm_D2.5mm_P7.62mm_Horizontal -> Resistor_SMD:R_1206_3216Metric_Pad1.30x1.75mm_HandSolder
- R14: renamed from R3; footprint Resistor_THT:R_Axial_DIN0207_L6.3mm_D2.5mm_P7.62mm_Horizontal -> Resistor_SMD:R_1206_3216Metric_Pad1.30x1.75mm_HandSolder
- R16: renamed from R6; footprint Resistor_THT:R_Axial_DIN0207_L6.3mm_D2.5mm_P7.62mm_Horizontal -> Resistor_SMD:R_1206_3216Metric_Pad1.30x1.75mm_HandSolder
- R19: renamed from R8; footprint Resistor_THT:R_Axial_DIN0207_L6.3mm_D2.5mm_P7.62mm_Horizontal -> Resistor_SMD:R_1206_3216Metric_Pad1.30x1.75mm_HandSolder
- R3: renamed from R2; footprint Resistor_THT:R_Axial_DIN0207_L6.3mm_D2.5mm_P7.62mm_Horizontal -> Resistor_SMD:R_1206_3216Metric_Pad1.30x1.75mm_HandSolder
- R6: renamed from R5; footprint Resistor_THT:R_Axial_DIN0207_L6.3mm_D2.5mm_P7.62mm_Horizontal -> Resistor_SMD:R_1206_3216Metric_Pad1.30x1.75mm_HandSolder
- R8: renamed from R7; footprint Resistor_THT:R_Axial_DIN0207_L6.3mm_D2.5mm_P7.62mm_Horizontal -> Resistor_SMD:R_1206_3216Metric_Pad1.30x1.75mm_HandSolder
- RV1, RV3: footprint noise_floor:Potentiometer_Single_3_Horizontal -> noise_floor:Potentiometer_Alpha_RD901F-40-00D_Single_Vertical_with_3DModel_from_Vasily_Kashirin
- RV5: renamed from RV2; footprint noise_floor:Potentiometer_Single_3_Horizontal -> noise_floor:Potentiometer_Alpha_RD901F-40-00D_Single_Vertical_with_3DModel_from_Vasily_Kashirin
- moved R3 39.7 mm to (57.6, 99.5)
- moved RV1 35.8 mm to (60.1, 101.5), turned to 90 degrees
- moved R1 34.7 mm to (59.1, 95.9), turned to 90 degrees
- moved R6 34.6 mm to (56.0, 95.9), turned to 90 degrees
- moved SW4 32.0 mm to (22.9, 124.7)
- moved SW2 32.0 mm to (59.1, 124.7)
- moved R19 24.6 mm to (22.9, 95.9), turned to 90 degrees
- moved R16 22.3 mm to (24.4, 99.5), turned to 0 degrees
- moved J4 20.5 mm to (32.7, 118.9)
- moved J11 20.4 mm to (49.3, 118.9)
- moved R10 19.9 mm to (41.0, 99.5)
- moved R12 18.5 mm to (39.5, 95.9), turned to 90 degrees
- moved R8 18.5 mm to (42.5, 95.9), turned to 90 degrees
- moved RV3 15.2 mm to (43.5, 101.5), turned to 90 degrees
- moved RV5 14.6 mm to (26.9, 101.5), turned to 90 degrees
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- renumbered J11 to J10, J6 to J5, J7 to J6, J8 to J7, J9 to J8, J10 to J9, R11 to R18, R4 to R5
Connections:
- J11 pad 1: unconnected-(J5-Pin_1-Pad1) -> /POT5_CCW
- J11 pad 11: /SPDT3_NO -> unconnected-(J11-Pin_11-Pad11)
- J11 pad 13: /SPDT3_COM -> unconnected-(J11-Pin_13-Pad13)
- J11 pad 14: /GND_UX -> /POT1_CW
- J11 pad 15: /SPDT3_NC -> /POT1_WIPER
- J11 pad 18: (no net) -> /GND_UX
- J11 pad 19: (no net) -> /GND_UX
- J11 pad 2: /POT2_CCW -> /POT5_WIPER
- J11 pad 3: unconnected-(J5-Pin_3-Pad3) -> /POT5_CW
- J11 pad 4: /POT2_CW -> unconnected-(J11-Pin_4-Pad4)
- J11 pad 5: /SPDT2_NC -> unconnected-(J11-Pin_5-Pad5)
- J11 pad 6: /POT2_WIPER -> unconnected-(J11-Pin_6-Pad6)
- J11 pad 7: /SPDT2_COM -> unconnected-(J11-Pin_7-Pad7)
- J11 pad 9: /SPDT2_NO -> unconnected-(J11-Pin_9-Pad9)
- J4 pad 1: /SPDT1_NC -> /SPDT2_NO
- J4 pad 10: /POT1_WIPER -> unconnected-(J4-Pin_10-Pad10)
- J4 pad 11: /POT3_CW -> /POT2_CW
- J4 pad 12: /POT1_CCW -> /POT2_WIPER
- J4 pad 13: /POT3_WIPER -> /POT2_CCW
- J4 pad 14: /POT1_CW -> /SPDT3_NO
- J4 pad 15: /POT3_CCW -> /SPDT3_COM
- J4 pad 18: (no net) -> /POT6_WIPER
- J4 pad 19: (no net) -> /POT6_CCW
- J4 pad 2: /GND_UX -> /SPDT2_COM
- J4 pad 3: /SPDT1_COM -> /SPDT2_NC
- J4 pad 5: /SPDT1_NO -> unconnected-(J4-Pin_5-Pad5)
Routing:
- net /SPDT2_NO: track 34.4 -> 8.08 mm
- net /SPDT3_NO: track 34.2 -> 9.76 mm
- net /SPDT1_NO: track 34.2 -> 9.81 mm
- net /SPDT2_COM: track 30.6 -> 6.52 mm
- net /SPDT1_COM: track 28.2 -> 8.25 mm
- net /SPDT3_COM: track 28.1 -> 8.20 mm
- net /SPDT2_NC: track 26.9 -> 7.44 mm
- net /POT5_WIPER: track 0.00 -> 19.2 mm, vias 0 -> 1
- net /POT4_WIPER: track 0.00 -> 18.3 mm
- net /POT6_WIPER: track 0.00 -> 18.3 mm
- net /POT3_WIPER: track 43.2 -> 26.2 mm, vias 0 -> 1
- net /POT4_CCW: track 0.00 -> 15.7 mm
- net /POT6_CW: track 0.00 -> 15.6 mm
- net /SPDT3_NC: track 23.6 -> 8.71 mm
- net /POT5_CW: track 0.00 -> 14.5 mm
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